Commit message: Adding GPS to simulation, broken atm, gps.xacro needs to be rewritten

File: src/snowplow/description/gps.xacro (robot description, xacro)
@@ -2,49 +2,52 @@
 <robot xmlns:xacro="http://www.ros.org/wiki/xacro" >
   <joint name="gps_joint" type="fixed">
-    <parent link="chassis"/>
-    <child link="gps_link"/>
-    <origin xyz="0 0 0" rpy="0 0 0"/>
+    <parent>chassis</parent>
+    <child>gps_link</child>
+    <pose>-0.05 0 0.05 0 0 0</pose>
+    <axis>
+      <xyz>0 0 1</xyz>
+    </axis>
   </joint>
   <link name="gps_link">
-      <!-- Some weird bug occurs if this joint gets the default inertia -->
-        <inertial>
-          <pose>-0.052 0 0.111 0 0 0</pose>
-          <inertia>
-            <mass>0.001</mass>
-            <ixx>0.001</ixx>
-            <ixy>0.000</ixy>
-            <ixz>0.000</ixz>
-            <iyy>0.001</iyy>
-            <iyz>0.000</iyz>
-            <izz>0.001</izz>
-          </inertia>
-          <mass>0.125</mass>
-        </inertial>
-        <sensor name="snowplow_gps" type="gps">
-          <always_on>true</always_on>
-          <update_rate>1</update_rate>
-          <pose>0 0 0 0 0 0</pose>
-          <gps>
-            <position_sensing>
-              <horizontal>
-                <noise type="gaussian">
-                  <mean>0.0</mean>
-                  <stddev>0.01</stddev>
-                </noise>
-              </horizontal>
-              <vertical>
-                <noise type="gaussian">
-                  <mean>0.0</mean>
-                  <stddev>0.01</stddev>
-                </noise>
-              </vertical>
-            </position_sensing>
-          </gps>
-          <plugin name="my_gps_plugin" filename="libgazebo_ros_gps_sensor.so">
-            <ros>
-              <remapping>~/out:=/gps/fix</remapping>
-            </ros>
-          </plugin>
-        </sensor>
-      </link>
+  <!-- Some weird bug occurs if this joint gets the default inertia -->
+    <inertial>
+      <pose>-0.052 0 0.111 0 0 0</pose>
+      <inertia>
+        <mass>0.001</mass>
+        <ixx>0.001</ixx>
+        <ixy>0.000</ixy>
+        <ixz>0.000</ixz>
+        <iyy>0.001</iyy>
+        <iyz>0.000</iyz>
+        <izz>0.001</izz>
+      </inertia>
+      <mass>0.125</mass>
+    </inertial>
+    <sensor name="snowplow_gps" type="gps">
+      <always_on>true</always_on>
+      <update_rate>1</update_rate>
+      <pose>0 0 0 0 0 0</pose>
+      <gps>
+        <position_sensing>
+          <horizontal>
+            <noise type="gaussian">
+              <mean>0.0</mean>
+              <stddev>0.01</stddev>
+            </noise>
+          </horizontal>
+          <vertical>
+            <noise type="gaussian">
+              <mean>0.0</mean>
+              <stddev>0.01</stddev>
+            </noise>
+          </vertical>
+        </position_sensing>
+      </gps>
+      <plugin name="my_gps_plugin" filename="libgazebo_ros_gps_sensor.so">
+        <ros>
+          <remapping>~/out:=/gps/fix</remapping>
+        </ros>
+      </plugin>
+    </sensor>
+  </link>
 </robot>

File: src/snowplow/description/lidar.xacro (robot description, xacro)
@@ -50,5 +50,5 @@
             <plugin name="laser_controller" filename="libgazebo_ros_ray_sensor.so">
                 <ros>
-                    <argument>~/out:=scan</argument>
+                    <argument>--ros-args --remap ~/out:=scan</argument>
                 </ros>
                 <output_type>sensor_msgs/LaserScan</output_type>

File: src/snowplow/description/robot.urdf.xacro (robot description, xacro)
@@ -12,4 +12,5 @@
     <xacro:include filename="lidar.xacro" />
     <xacro:include filename="imu.xacro" />
+    <xacro:include filename="gps.xacro"/>
     <!-- <xacro:include filename="camera.xacro" /> -->
     <!-- <xacro:include filename="depth_camera.xacro" /> -->

Commit message: Attempting to fix gps plugin. frames are fixed but plugin still doesn't work

File: src/snowplow/description/gps.xacro (robot description, xacro)
@@ -2,31 +2,24 @@
 <robot xmlns:xacro="http://www.ros.org/wiki/xacro" >
   <joint name="gps_joint" type="fixed">
-    <parent>chassis</parent>
-    <child>gps_link</child>
-    <pose>-0.05 0 0.05 0 0 0</pose>
-    <axis>
-      <xyz>0 0 1</xyz>
-    </axis>
+    <parent link="chassis"/>
+    <child link="gps_link"/>
+    <origin xyz="0.276 0 0" rpy="0 0.18 0"/>
   </joint>
   <link name="gps_link">
-  <!-- Some weird bug occurs if this joint gets the default inertia -->
-    <inertial>
-      <pose>-0.052 0 0.111 0 0 0</pose>
-      <inertia>
-        <mass>0.001</mass>
-        <ixx>0.001</ixx>
-        <ixy>0.000</ixy>
-        <ixz>0.000</ixz>
-        <iyy>0.001</iyy>
-        <iyz>0.000</iyz>
-        <izz>0.001</izz>
-      </inertia>
-      <mass>0.125</mass>
-    </inertial>
-    <sensor name="snowplow_gps" type="gps">
-      <always_on>true</always_on>
-      <update_rate>1</update_rate>
-      <pose>0 0 0 0 0 0</pose>
-      <gps>
+    <visual>
+      <geometry>
+          <box size="0.010 0.01 0.01"/>
+      </geometry>
+      <material name="black"/>
+    </visual>
+  </link>
+  <gazebo reference="gps_link">
+      <material>Gazebo/Black</material>
+      <gravity>true</gravity>
+      <sensor name="snowplow_gps" type="gps">
+        <always_on>true</always_on>
+        <update_rate>1</update_rate>
+        <pose>0 0 0 0 0 0</pose>
+        <gps>
         <position_sensing>
           <horizontal>
@@ -44,10 +37,28 @@
         </position_sensing>
       </gps>
-      <plugin name="my_gps_plugin" filename="libgazebo_ros_gps_sensor.so">
+      <!-- <plugin name="my_gps_plugin" filename="libgazebo_ros_gps_sensor.so">
         <ros>
+          <namespace>/gps</namespace>
           <remapping>~/out:=/gps/fix</remapping>
         </ros>
+        <frame_name>gps_link</frame_name>
+      </plugin> -->
+      <plugin name="hector_gps" filename="libgazebo_ros_gps.so">
+        <alwaysOn>true</alwaysOn>
+        <updateRate>30.0</updateRate>
+        <bodyName>chassis</bodyName>
+        <frameId>gps_link</frameId>
+        <topicName>/fix</topicName>
+        <velocityTopicName>/fix_vel</velocityTopicName>
+        <!-- <referenceLatitude>50.090337</referenceLatitude> -->
+        <!-- <referenceLongitude>14.133275</referenceLongitude> -->
+        <referenceLatitude>0.0</referenceLatitude>
+        <referenceLongitude>0.0</referenceLongitude>
+        <drift>0.0001 0.0001 0.0001</drift>
+        <gaussianNoise>0.0 0.0 0.0</gaussianNoise>
+        <velocityDrift>0 0 0</velocityDrift>
+        <velocityGaussianNoise>0.0 0.0 0.0</velocityGaussianNoise>
       </plugin>
     </sensor>
-  </link>
+  </gazebo>
 </robot>
