Commit message: Fixing friction slipping issues (Still some slippage)

File: src/snowplow/description/battery.xacro (robot description, xacro)
@@ -20,5 +20,5 @@
             </geometry>
         </collision>
-        <xacro:inertial_box mass="30.0" x="${chassis_length/2}" y="${chassis_width/2}" z="${chassis_height/2}">
+        <xacro:inertial_box mass="2.0" x="${chassis_length/2}" y="${chassis_width/2}" z="${chassis_height/2}">
             <origin xyz="0 0 0" rpy="0 0 0"/>
         </xacro:inertial_box>

File: src/snowplow/description/lidar.xacro (robot description, xacro)
@@ -5,5 +5,5 @@
         <parent link="chassis"/>
         <child link="laser_frame"/>
-        <origin xyz="0.10 0 0.556" rpy="0 0 0"/>
+        <origin xyz="0.10 0 0.66" rpy="0 0 0"/>
     </joint>
     <link name="laser_frame">
@@ -15,5 +15,5 @@
         </visual>
         <visual>
-            <origin xyz="0 0 -0.05"/>
+            <origin xyz="0 0 0"/>
             <geometry>
                 <cylinder radius="0.07" length="0.1"/>
@@ -40,5 +40,6 @@
                     <horizontal>
                         <samples>360</samples>
-                        <min_angle>-3.14</min_angle>
+                        <min_angle>0</min_angle>
+                        <!-- <min_angle>-3.14</min_angle> -->
                         <max_angle>3.14</max_angle>
                     </horizontal>
@@ -62,5 +63,5 @@
         <parent link="chassis"/>
         <child link="lidar_holder"/>
-        <origin xyz="0 0 0.456" rpy="0 0 0"/>
+        <origin xyz="0 0 0.466" rpy="0 0 0"/>
     </joint>
     <link name="lidar_holder">
@@ -76,5 +77,5 @@
             </geometry>
         </collision>
-        <xacro:inertial_box mass="0.05" x="0.25" y="0.14" z="0.03">
+        <xacro:inertial_box mass="0.01" x="0.25" y="0.14" z="0.03">
             <origin xyz="0 0 0" rpy="0 0 0"/>
         </xacro:inertial_box>

File: src/snowplow/description/plowblade.xacro (robot description, xacro)
@@ -2,5 +2,5 @@
 <robot xmlns:xacro="http://ros.org/wiki/xacro">
   <!-- Define parameters -->
-    <xacro:property name="plow_height" value="${chassis_height - 0.2}"/> <!-- Height of the snowplow blade -->
+  <xacro:property name="plow_height" value="${chassis_height - 0.2}"/> <!-- Height of the snowplow blade -->
   <xacro:property name="plow_width" value="1.5"/> <!-- Width of the snowplow blade -->
   <xacro:property name="plow_length" value="0.1"/> <!-- Length of the snowplow blade -->
@@ -27,5 +27,5 @@
         <collision>
             <geometry>
-                <cylinder radius="0.01"/>
+                <cylinder radius="0.01" length="${bar_length}"/>
             </geometry>
         </collision>
@@ -79,8 +79,7 @@
   <!-- Gazebo specific properties -->
   <gazebo reference="snowplow_blade_link">
-    <mu1>1000</mu1> <!-- Friction coefficient -->
-    <mu2>1000</mu2> <!-- Friction coefficient -->
+    <!-- <mu1>1000</mu1> Friction coefficient -->
+    <!-- <mu2>1000</mu2> Friction coefficient -->
     <material>Gazebo/Grey</material> <!-- Gazebo built-in material -->
-    <turnGravityOff>true</turnGravityOff> <!-- Turn off gravity for the link -->
   </gazebo>
 </robot>

File: src/snowplow/description/robot_core.xacro (robot description, xacro)
@@ -5,13 +5,13 @@
     <xacro:property name="chassis_width" value="0.696"/>
     <xacro:property name="chassis_height" value="0.556"/>
-    <xacro:property name="chassis_mass" value="1.0"/>
+    <xacro:property name="chassis_mass" value="3.0"/>
     <xacro:property name="wheel_radius" value="0.16"/>
     <xacro:property name="wheel_thickness" value="0.19"/>
-    <xacro:property name="wheel_mass" value="0.05"/>
+    <xacro:property name="wheel_mass" value="1.0"/>
     <xacro:property name="wheel_offset_x" value="0.226"/>
     <xacro:property name="wheel_offset_y" value="${chassis_width/2 + wheel_thickness + 0.01}"/>
     <xacro:property name="wheel_offset_z" value="0.01"/>
     <xacro:property name="caster_wheel_radius" value="0.01"/>
-    <xacro:property name="caster_wheel_mass" value="0.01"/>
+    <xacro:property name="caster_wheel_mass" value="0.2"/>
     <xacro:property name="caster_wheel_offset_x" value="0.075"/>
     <xacro:property name="caster_wheel_offset_z" value="${wheel_offset_z - wheel_radius + caster_wheel_radius}"/>
@@ -71,5 +71,5 @@
             </geometry>
         </collision>
-        <xacro:inertial_box mass="0.5" x="${chassis_length}" y="${chassis_width}" z="${chassis_height}">
+        <xacro:inertial_box mass="${chassis_mass}" x="${chassis_length}" y="${chassis_width}" z="${chassis_height}">
             <origin xyz="${-chassis_length/2} 0 ${chassis_height/2}" rpy="0 0 0"/>
         </xacro:inertial_box>
@@ -129,4 +129,6 @@
     <gazebo reference="right_wheel">
         <material>Gazebo/Black</material>
+        <!-- <mu1>0.01</mu1>
+        <mu2>0.01</mu2>  -->
     </gazebo>
     <joint name="wheel_joint" type="fixed">
@@ -145,5 +147,5 @@
         <collision>
             <geometry>
-                <cylinder radius="0.01"/>
+                <cylinder radius="0.01" length="${chassis_width + wheel_thickness + 0.01}"/>
             </geometry>
         </collision>

Commit message: Fixing mass and inertial issues of the robot

File: src/snowplow/description/battery.xacro (robot description, xacro)
@@ -20,6 +20,6 @@
             </geometry>
         </collision>
-        <xacro:inertial_box mass="2.0" x="${chassis_length/2}" y="${chassis_width/2}" z="${chassis_height/2}">
-            <origin xyz="0 0 0" rpy="0 0 0"/>
+        <xacro:inertial_box mass="2.0" x="0.3" y="0.5" z="0.3">
+            <origin xyz="${chassis_length/2} ${chassis_width/2} -0.5" rpy="0 0 0"/>
         </xacro:inertial_box>
     </link>

File: src/snowplow/description/gazebo_control.xacro (robot description, xacro)
@@ -10,5 +10,5 @@
             <!-- Limits -->
             <max_wheel_torque>200</max_wheel_torque>
-            <max_wheel_acceleration>10.0</max_wheel_acceleration>
+            <max_wheel_acceleration>5.0</max_wheel_acceleration>
             <!-- Output -->
             <odometry_frame>odom</odometry_frame>

File: src/snowplow/description/plowblade.xacro (robot description, xacro)
@@ -76,9 +76,10 @@
       </geometry>
     </collision>
+    <xacro:inertial_box mass="1.0" x="${plow_length}" y="${plow_width}" z="${plow_height}">
+      <origin xyz="${plow_length / 2} 0 -0.01" rpy="0 0 0"/>
+    </xacro:inertial_box>
   </link>
   <!-- Gazebo specific properties -->
   <gazebo reference="snowplow_blade_link">
-    <!-- <mu1>1000</mu1> Friction coefficient -->
-    <!-- <mu2>1000</mu2> Friction coefficient -->
     <material>Gazebo/Grey</material> <!-- Gazebo built-in material -->
   </gazebo>

File: src/snowplow/description/robot_core.xacro (robot description, xacro)
@@ -96,4 +96,17 @@
                 <sphere radius="${wheel_radius}"/>
             </geometry>
+            <surface>
+                <friction>
+                <ode>
+                    <mu>10000.0</mu>
+                    <mu2>10000.0</mu2>
+                </ode>
+                </friction>
+                <contact>
+                <ode>
+                    <min_depth>0.003</min_depth>
+                </ode>
+                </contact>
+            </surface>
         </collision>
         <xacro:inertial_cylinder mass="${wheel_mass}" length="${wheel_thickness}" radius="${wheel_radius}">
@@ -122,4 +135,17 @@
                 <sphere radius="${wheel_radius}"/>
             </geometry>
+            <surface>
+                <friction>
+                <ode>
+                    <mu>10000.0</mu>
+                    <mu2>10000.0</mu2>
+                </ode>
+                </friction>
+                <contact>
+                <ode>
+                    <min_depth>0.003</min_depth>
+                </ode>
+                </contact>
+            </surface>
         </collision>
         <xacro:inertial_cylinder mass="${wheel_mass}" length="${wheel_thickness}" radius="${wheel_radius}">
@@ -129,6 +155,4 @@
     <gazebo reference="right_wheel">
         <material>Gazebo/Black</material>
-        <!-- <mu1>0.01</mu1>
-        <mu2>0.01</mu2>  -->
     </gazebo>
     <joint name="wheel_joint" type="fixed">

File: src/snowplow/description/ros2_control.xacro (robot description, xacro)
@@ -38,6 +38,6 @@
             <joint name="left_wheel_joint">
                 <command_interface name="velocity">
-                    <param name="min">-10</param>
-                    <param name="max">10</param>
+                    <param name="min">-2</param>
+                    <param name="max">2</param>
                 </command_interface>
                 <state_interface name="velocity"/>
@@ -46,6 +46,6 @@
             <joint name="right_wheel_joint">
                 <command_interface name="velocity">
-                    <param name="min">-10</param>
-                    <param name="max">10</param>
+                    <param name="min">-2</param>
+                    <param name="max">2</param>
                 </command_interface>
                 <state_interface name="velocity"/>
