Commit message: Broken build atm, trying different things...

File: src/snowplow/description/robot.urdf_ign.xacro (robot description, xacro)
@@ -5,5 +5,5 @@
     <xacro:include filename="$(find snowplow)/description/robot_core.xacro" />
     <!-- <xacro:if value="$(arg use_ros2_control)"> -->
-        <xacro:include filename="$(find snowplow)/description/ros2_control_ign.xacro" />
+    <xacro:include filename="$(find snowplow)/description/ros2_control_ign.xacro" />
     <!-- </xacro:if> -->
     <xacro:include filename="$(find snowplow)/description/lidar_ign.xacro" />
@@ -11,5 +11,5 @@
     <xacro:include filename="$(find snowplow)/description/gps_ign.xacro"/>
     <xacro:include filename="$(find snowplow)/description/plowblade.xacro"/>
-    <xacro:include filename="$(find snowplow)/description/battery.xacro"/>
+    <!-- <xacro:include filename="$(find snowplow)/description/battery.xacro"/> -->
     <!-- <xacro:include filename="camera.xacro" /> -->
     <!-- <xacro:include filename="depth_camera.xacro" /> -->

File: src/snowplow/description/robot_core.xacro (robot description, xacro)
@@ -202,6 +202,6 @@
     <gazebo reference="caster_wheel">
         <material>Gazebo/White</material>
-        <mu1 value="0.001"/>
-        <mu2 value="0.001"/>
+        <mu1 value="0.000"/>
+        <mu2 value="0.000"/>
     </gazebo>
 </robot>

File: src/snowplow/description/ros2_control_ign.xacro (robot description, xacro)
@@ -1,58 +1,25 @@
 <?xml version="1.0"?>
 <robot xmlns:xacro="http://www.ros.org/wiki/xacro">
-    <xacro:unless value="$(arg use_sim_time)">
-        <ros2_control name="RealRobot" type="system">
-            <hardware>
-                <plugin>motor_controller/DiffBotSystemHardware</plugin>
-                <param name="left_wheel_name">left_wheel_joint</param>
-                <param name="right_wheel_name">right_wheel_joint</param>
-                <param name="loop_rate">30</param>
-                <param name="device">/dev/ttyUSB0</param>
-                <param name="baud_rate">115200</param>
-                <param name="timeout">1000</param>
-                <!-- Check the enc counter parameter with the electrical team -->
-                <param name="enc_counts_per_rev">3000</param>
-            </hardware>
-            <joint name="left_wheel_joint">
-                <command_interface name="velocity">
-                    <param name="min">-10</param>
-                    <param name="max">10</param>
-                </command_interface>
-                <state_interface name="velocity"/>
-                <state_interface name="position"/>
-            </joint>
-            <joint name="right_wheel_joint">
-                <command_interface name="velocity">
-                    <param name="min">-10</param>
-                    <param name="max">10</param>
-                </command_interface>
-                <state_interface name="velocity"/>
-                <state_interface name="position"/>
-            </joint>
-        </ros2_control>
-    </xacro:unless>
-    <xacro:if value="$(arg use_sim_time)">
-        <ros2_control name="IgnitionSystem" type="system">
-            <hardware>
-                <plugin>ign_ros2_control/IgnitionSystem</plugin>
-            </hardware>
-            <joint name="left_wheel_joint">
-                <command_interface name="velocity">
-                    <param name="min">-2</param>
-                    <param name="max">2</param>
-                </command_interface>
-                <state_interface name="velocity"/>
-                <state_interface name="position"/>
-            </joint>
-            <joint name="right_wheel_joint">
-                <command_interface name="velocity">
-                    <param name="min">-2</param>
-                    <param name="max">2</param>
-                </command_interface>
-                <state_interface name="velocity"/>
-                <state_interface name="position"/>
-            </joint>
-        </ros2_control>
-    </xacro:if>
+    <ros2_control name="IgnitionSystem" type="system">
+        <hardware>
+            <plugin>ign_ros2_control/IgnitionSystem</plugin>
+        </hardware>
+        <joint name="left_wheel_joint">
+            <command_interface name="velocity">
+                <param name="min">-2</param>
+                <param name="max">2</param>
+            </command_interface>
+            <state_interface name="velocity"/>
+            <state_interface name="position"/>
+        </joint>
+        <joint name="right_wheel_joint">
+            <command_interface name="velocity">
+                <param name="min">-2</param>
+                <param name="max">2</param>
+            </command_interface>
+            <state_interface name="velocity"/>
+            <state_interface name="position"/>
+        </joint>
+    </ros2_control>
     <gazebo>
         <plugin filename="ign_ros2_control-system" name="ign_ros2_control::IgnitionROS2ControlPlugin">
@@ -60,7 +27,4 @@
             <!-- <controller_manager_name>controller_manager</controller_manager_name> -->
         </plugin>
-        <plugin name="motor_controller" filename="libmotor_controller.so">
-            <parameters>$(find snowplow)/config/my_controllers.yaml</parameters>
-        </plugin>
     </gazebo>
 </robot>

Commit message: Fixing launch and simplifying urdf

File: src/snowplow/description/robot.urdf_ign.xacro (robot description, xacro)
@@ -4,7 +4,5 @@
     <xacro:arg name="use_sim_time" default="true"/>
     <xacro:include filename="$(find snowplow)/description/robot_core.xacro" />
-    <!-- <xacro:if value="$(arg use_ros2_control)"> -->
-        <xacro:include filename="$(find snowplow)/description/ros2_control_ign.xacro" />
-    <!-- </xacro:if> -->
+    <xacro:include filename="$(find snowplow)/description/ros2_control_ign.xacro" />
     <xacro:include filename="$(find snowplow)/description/lidar_ign.xacro" />
     <xacro:include filename="$(find snowplow)/description/imu_ign.xacro" />

File: src/snowplow/description/robot_core.xacro (robot description, xacro)
@@ -84,4 +84,5 @@
         <origin xyz="0 ${wheel_offset_y} 0" rpy="-${pi/2} 0 0" />
         <axis xyz="0 0 1"/>
+        <dynamics damping="0.2"/>
     </joint>
     <link name="left_wheel">

File: src/snowplow/description/ros2_control_ign.xacro (robot description, xacro)
@@ -1,58 +1,25 @@
 <?xml version="1.0"?>
 <robot xmlns:xacro="http://www.ros.org/wiki/xacro">
-    <xacro:unless value="$(arg use_sim_time)">
-        <ros2_control name="RealRobot" type="system">
-            <hardware>
-                <plugin>motor_controller/DiffBotSystemHardware</plugin>
-                <param name="left_wheel_name">left_wheel_joint</param>
-                <param name="right_wheel_name">right_wheel_joint</param>
-                <param name="loop_rate">30</param>
-                <param name="device">/dev/ttyUSB0</param>
-                <param name="baud_rate">115200</param>
-                <param name="timeout">1000</param>
-                <!-- Check the enc counter parameter with the electrical team -->
-                <param name="enc_counts_per_rev">3000</param>
-            </hardware>
-            <joint name="left_wheel_joint">
-                <command_interface name="velocity">
-                    <param name="min">-10</param>
-                    <param name="max">10</param>
-                </command_interface>
-                <state_interface name="velocity"/>
-                <state_interface name="position"/>
-            </joint>
-            <joint name="right_wheel_joint">
-                <command_interface name="velocity">
-                    <param name="min">-10</param>
-                    <param name="max">10</param>
-                </command_interface>
-                <state_interface name="velocity"/>
-                <state_interface name="position"/>
-            </joint>
-        </ros2_control>
-    </xacro:unless>
-    <xacro:if value="$(arg use_sim_time)">
-        <ros2_control name="IgnitionSystem" type="system">
-            <hardware>
-                <plugin>ign_ros2_control/IgnitionSystem</plugin>
-            </hardware>
-            <joint name="left_wheel_joint">
-                <command_interface name="velocity">
-                    <param name="min">-2</param>
-                    <param name="max">2</param>
-                </command_interface>
-                <state_interface name="velocity"/>
-                <state_interface name="position"/>
-            </joint>
-            <joint name="right_wheel_joint">
-                <command_interface name="velocity">
-                    <param name="min">-2</param>
-                    <param name="max">2</param>
-                </command_interface>
-                <state_interface name="velocity"/>
-                <state_interface name="position"/>
-            </joint>
-        </ros2_control>
-    </xacro:if>
+    <ros2_control name="IgnitionSystem" type="system">
+        <hardware>
+            <plugin>ign_ros2_control/IgnitionSystem</plugin>
+        </hardware>
+        <joint name="left_wheel_joint">
+            <command_interface name="velocity">
+                <param name="min">-5</param>
+                <param name="max">5</param>
+            </command_interface>
+            <state_interface name="velocity"/>
+            <state_interface name="position"/>
+        </joint>
+        <joint name="right_wheel_joint">
+            <command_interface name="velocity">
+                <param name="min">-5</param>
+                <param name="max">5</param>
+            </command_interface>
+            <state_interface name="velocity"/>
+            <state_interface name="position"/>
+        </joint>
+    </ros2_control>
     <gazebo>
         <plugin filename="ign_ros2_control-system" name="ign_ros2_control::IgnitionROS2ControlPlugin">
