Commit message: FIXED ALL ROS2 CONTROL ISSUES!

File: src/snowplow/description/robot_core.xacro (robot description, xacro)
@@ -201,8 +201,3 @@
         </xacro:inertial_sphere>
     </link>
-    <gazebo reference="caster_wheel">
-        <material>Gazebo/White</material>
-        <mu1 value="0.001"/>
-        <mu2 value="0.001"/>
-    </gazebo>
 </robot>

File: src/snowplow/description/ros2_control_ign.xacro (robot description, xacro)
@@ -27,7 +27,4 @@
             <!-- <controller_manager_name>controller_manager</controller_manager_name> -->
         </plugin>
-        <plugin name="motor_controller" filename="libmotor_controller.so">
-            <parameters>$(find snowplow)/config/my_controllers.yaml</parameters>
-        </plugin>
     </gazebo>
 </robot>
