Commit message: Fixing jitter issues

File: src/snowplow/description/imu_ign.xacro (robot description, xacro)
@@ -4,5 +4,5 @@
         <parent link="chassis"/>
         <child link="imu_link"/>
-        <origin xyz="-0.375 0 0.278" rpy="0 0.18 0"/>
+        <origin xyz="-0.675 0 0.278" rpy="0 0.0 0"/>
     </joint>
     <link name="imu_link">
@@ -29,5 +29,5 @@
             <sensor name="imu" type="imu">
             <always_on>1</always_on>
-            <update_rate>10</update_rate> <!-- To simulate orientation coming from dual GNSS -->
+            <update_rate>25</update_rate> <!-- To simulate orientation coming from dual GNSS -->
             <visualize>false</visualize>
             <topic>imu</topic>

File: src/snowplow/description/lidar_ign.xacro (robot description, xacro)
@@ -40,9 +40,10 @@
         <gazebo reference="laser_frame">
             <material>Gazebo/Black</material>
+            <ignition_frame_id>laser_frame</ignition_frame_id>
             <sensor name="gpu_lidar" type="gpu_lidar">
-                <pose relative_to='laser_frame'> 0 0 0 0 0 4.713 </pose>
+                <pose relative_to='laser_frame'> 0 0 0 0 0 4.71 </pose>
                 <topic>scan</topic>
                 <visualize>true</visualize>
-                <update_rate>5</update_rate>
+                <update_rate>20</update_rate>
                 <ray>
                     <scan>
@@ -50,6 +51,6 @@
                             <samples>360</samples>
                             <min_angle>0</min_angle>
-                            <min_angle>-3.14</min_angle>
-                            <max_angle>3.14</max_angle>
+                            <min_angle>0</min_angle>
+                            <max_angle>6.283</max_angle>
                         </horizontal>
                     </scan>

Commit message: Fixed a lot of things (jitter, parameter configs, launch, urdf)

File: src/snowplow/description/imu_ign.xacro (robot description, xacro)
@@ -4,20 +4,16 @@
         <parent link="chassis"/>
         <child link="imu_link"/>
-        <origin xyz="-0.675 0 0.278" rpy="0 0.0 0"/>
+        <origin xyz="0.675 0 1.0" rpy="0 0.0 0"/>
     </joint>
     <link name="imu_link">
         <visual>
             <geometry>
-                <box size="0.07 0.03 0.03"/>
+                <box size="0.046 0.045 0.024"/>
             </geometry>
             <material name="black"/>
         </visual>
-        <visual>
-            <origin xyz="0 0 -0.05"/>
-            <geometry>
-                <cylinder radius="0.002" length="0.1"/>
-            </geometry>
-            <material name="black"/>
-        </visual>
+        <xacro:inertial_box mass="0.029" x="0.046" y="0.045" z="0.024">
+            <origin xyz="0 0 0" rpy="0 0 0"/>
+        </xacro:inertial_box>
     </link>
     <!-- Only enable gazebo simulation if in simulation mode -->
@@ -28,9 +24,9 @@
         <gazebo reference="imu_link">
             <sensor name="imu" type="imu">
-            <always_on>1</always_on>
-            <update_rate>25</update_rate> <!-- To simulate orientation coming from dual GNSS -->
-            <visualize>false</visualize>
-            <topic>imu</topic>
-            <ignition_frame_id>imu_link</ignition_frame_id>
+                    <always_on>1</always_on>
+                    <update_rate>25</update_rate> <!-- To simulate orientation coming from dual GNSS -->
+                    <visualize>false</visualize>
+                    <topic>imu</topic>
+                    <ignition_frame_id>imu_link</ignition_frame_id>
             </sensor>
         </gazebo>

File: src/snowplow/description/lidar_ign.xacro (robot description, xacro)
@@ -40,6 +40,6 @@
         <gazebo reference="laser_frame">
             <material>Gazebo/Black</material>
-            <ignition_frame_id>laser_frame</ignition_frame_id>
             <sensor name="gpu_lidar" type="gpu_lidar">
+                <ignition_frame_id>laser_frame</ignition_frame_id>
                 <pose relative_to='laser_frame'> 0 0 0 0 0 4.71 </pose>
                 <topic>scan</topic>

File: src/snowplow/description/robot.urdf_ign.xacro (robot description, xacro)
@@ -8,5 +8,5 @@
     <xacro:include filename="$(find snowplow)/description/gps_ign.xacro"/>
     <xacro:include filename="$(find snowplow)/description/plowblade.xacro"/>
-    <xacro:include filename="$(find snowplow)/description/battery.xacro"/>
+    <!-- <xacro:include filename="$(find snowplow)/description/battery.xacro"/>  -->
     <xacro:include filename="$(find snowplow)/description/face.xacro" />
 </robot>

File: src/snowplow/description/robot_core.xacro (robot description, xacro)
@@ -183,5 +183,5 @@
         <parent link="chassis"/>
         <child link="caster_wheel"/>
-        <origin xyz="${-chassis_length + 0.1} 0 ${-wheel_radius/2}"/>
+        <origin xyz="${-chassis_length + 0.1} 0 ${-wheel_radius/2 + 0.01}"/>
     </joint>
     <link name="caster_wheel">

Commit message: wip

File: src/snowplow/description/imu_ign.xacro (robot description, xacro)
@@ -4,5 +4,5 @@
         <parent link="chassis"/>
         <child link="imu_link"/>
-        <origin xyz="0.675 0 1.0" rpy="0 0.0 0"/>
+        <origin xyz="0.475 0 0.5" rpy="0 0.0 0"/>
     </joint>
     <link name="imu_link">

File: src/snowplow/description/lidar_ign.xacro (robot description, xacro)
@@ -42,5 +42,5 @@
             <sensor name="gpu_lidar" type="gpu_lidar">
                 <ignition_frame_id>laser_frame</ignition_frame_id>
-                <pose relative_to='laser_frame'> 0 0 0 0 0 4.71 </pose>
+                <pose relative_to='laser_frame'> 0 0 0 0 0 0 </pose>
                 <topic>scan</topic>
                 <visualize>true</visualize>
