Commit message: Updating readme + changing launch structure

File: src/snowplow/description/gps_ign.xacro (robot description, xacro)
@@ -15,15 +15,17 @@
   </link>
   <!-- <gazebo> -->
-  <gazebo>
-      <plugin filename="ignition-gazebo-navsat-system" name="ignition::gazebo::systems::NavSat"/>
-  </gazebo>
-  <gazebo reference="gps_link">
-      <material>Gazebo/Black</material>
-      <sensor name="navsat" type="navsat">
-            <always_on>1</always_on>
-            <update_rate>25.0</update_rate>
-            <topic>gps/fix</topic>
-            <ignition_frame_id>gps_link</ignition_frame_id>
-      </sensor>
-  </gazebo>
+  <xacro:if value="$(arg use_sim_time)">
+    <gazebo>
+        <plugin filename="ignition-gazebo-navsat-system" name="ignition::gazebo::systems::NavSat"/>
+    </gazebo>
+    <gazebo reference="gps_link">
+        <material>Gazebo/Black</material>
+        <sensor name="navsat" type="navsat">
+              <always_on>1</always_on>
+              <update_rate>25.0</update_rate>
+              <topic>gps/fix</topic>
+              <ignition_frame_id>gps_link</ignition_frame_id>
+        </sensor>
+    </gazebo>
+  <xacro:if/>
 </robot>

File: src/snowplow/description/imu_ign.xacro (robot description, xacro)
@@ -21,15 +21,18 @@
         </visual>
     </link>
-    <gazebo>
-        <plugin filename="libignition-gazebo-imu-system.so" name="ignition::gazebo::systems::Imu"/>
-    </gazebo>
-    <gazebo reference="imu_link">
-        <sensor name="imu" type="imu">
-        <always_on>1</always_on>
-        <update_rate>10</update_rate> <!-- To simulate orientation coming from dual GNSS -->
-        <visualize>false</visualize>
-        <topic>imu</topic>
-        <ignition_frame_id>imu_link</ignition_frame_id>
-        </sensor>
-    </gazebo>
+    <!-- Only enable gazebo simulation if in simulation mode -->
+    <xacro:if value="$(arg use_sim_time)">
+        <gazebo>
+            <plugin filename="libignition-gazebo-imu-system.so" name="ignition::gazebo::systems::Imu"/>
+        </gazebo>
+        <gazebo reference="imu_link">
+            <sensor name="imu" type="imu">
+            <always_on>1</always_on>
+            <update_rate>10</update_rate> <!-- To simulate orientation coming from dual GNSS -->
+            <visualize>false</visualize>
+            <topic>imu</topic>
+            <ignition_frame_id>imu_link</ignition_frame_id>
+            </sensor>
+        </gazebo>
+    </xacro:if>
 </robot>

File: src/snowplow/description/lidar_ign.xacro (robot description, xacro)
@@ -30,35 +30,37 @@
         </xacro:inertial_cylinder>
     </link>
-    <gazebo>
-        <plugin
-        filename="libignition-gazebo-sensors-system.so"
-        name="ignition::gazebo::systems::Sensors">
-        <render_engine>ogre2</render_engine>
-        </plugin>
-    </gazebo>
-    <gazebo reference="laser_frame">
-        <material>Gazebo/Black</material>
-        <sensor name="gpu_lidar" type="gpu_lidar">
-            <pose relative_to='laser_frame'> 0 0 0 0 0 4.713 </pose>
-            <topic>scan</topic>
-            <visualize>true</visualize>
-            <update_rate>5</update_rate>
-            <ray>
-                <scan>
-                    <horizontal>
-                        <samples>360</samples>
-                        <min_angle>0</min_angle>
-                        <min_angle>-3.14</min_angle>
-                        <max_angle>3.14</max_angle>
-                    </horizontal>
-                </scan>
-                <range>
-                    <min>0.08</min>
-                    <max>20.0</max>
-                </range>
-            </ray>
-            <always_on>1</always_on>
-        </sensor>
-    </gazebo>
+    <xacro:if value="$(arg use_sim_time)">
+        <gazebo>
+            <plugin
+            filename="libignition-gazebo-sensors-system.so"
+            name="ignition::gazebo::systems::Sensors">
+            <render_engine>ogre2</render_engine>
+            </plugin>
+        </gazebo>
+        <gazebo reference="laser_frame">
+            <material>Gazebo/Black</material>
+            <sensor name="gpu_lidar" type="gpu_lidar">
+                <pose relative_to='laser_frame'> 0 0 0 0 0 4.713 </pose>
+                <topic>scan</topic>
+                <visualize>true</visualize>
+                <update_rate>5</update_rate>
+                <ray>
+                    <scan>
+                        <horizontal>
+                            <samples>360</samples>
+                            <min_angle>0</min_angle>
+                            <min_angle>-3.14</min_angle>
+                            <max_angle>3.14</max_angle>
+                        </horizontal>
+                    </scan>
+                    <range>
+                        <min>0.08</min>
+                        <max>20.0</max>
+                    </range>
+                </ray>
+                <always_on>1</always_on>
+            </sensor>
+        </gazebo>
+    </xacro:if>
     <!-- LIDAR HOLDER -->
     <joint name="mount_joint" type="fixed">

File: src/snowplow/description/ros2_control_ign.xacro (robot description, xacro)
@@ -1,29 +1,64 @@
 <?xml version="1.0"?>
 <robot xmlns:xacro="http://www.ros.org/wiki/xacro">
-    <ros2_control name="IgnitionSystem" type="system">
-        <hardware>
-            <plugin>ign_ros2_control/IgnitionSystem</plugin>
-        </hardware>
-        <joint name="left_wheel_joint">
-            <command_interface name="velocity">
-                <param name="min">-5</param>
-                <param name="max">5</param>
-            </command_interface>
-            <state_interface name="velocity"/>
-            <state_interface name="position"/>
-        </joint>
-        <joint name="right_wheel_joint">
-            <command_interface name="velocity">
-                <param name="min">-5</param>
-                <param name="max">5</param>
-            </command_interface>
-            <state_interface name="velocity"/>
-            <state_interface name="position"/>
-        </joint>
-    </ros2_control>
+    <xacro:unless value="$(arg use_sim_time)">
+        <ros2_control name="RealRobot" type="system">
+            <hardware>
+                <plugin>motor_controller/DiffBotSystemHardware</plugin>
+                <param name="left_wheel_name">left_wheel_joint</param>
+                <param name="right_wheel_name">right_wheel_joint</param>
+                <param name="loop_rate">30</param>
+                <param name="device">/dev/ttyUSB0</param>
+                <param name="baud_rate">115200</param>
+                <param name="timeout">1000</param>
+                <!-- Check the enc counter parameter with the electrical team -->
+                <param name="enc_counts_per_rev">3000</param>
+            </hardware>
+            <joint name="left_wheel_joint">
+                <command_interface name="velocity">
+                    <param name="min">-10</param>
+                    <param name="max">10</param>
+                </command_interface>
+                <state_interface name="velocity"/>
+                <state_interface name="position"/>
+            </joint>
+            <joint name="right_wheel_joint">
+                <command_interface name="velocity">
+                    <param name="min">-10</param>
+                    <param name="max">10</param>
+                </command_interface>
+                <state_interface name="velocity"/>
+                <state_interface name="position"/>
+            </joint>
+        </ros2_control>
+    </xacro:unless>
+    <xacro:if value="$(arg use_sim_time)">
+        <ros2_control name="IgnitionSystem" type="system">
+            <hardware>
+                <plugin>ign_ros2_control/IgnitionSystem</plugin>
+            </hardware>
+            <joint name="left_wheel_joint">
+                <command_interface name="velocity">
+                    <param name="min">-5</param>
+                    <param name="max">5</param>
+                </command_interface>
+                <state_interface name="velocity"/>
+                <state_interface name="position"/>
+            </joint>
+            <joint name="right_wheel_joint">
+                <command_interface name="velocity">
+                    <param name="min">-5</param>
+                    <param name="max">5</param>
+                </command_interface>
+                <state_interface name="velocity"/>
+                <state_interface name="position"/>
+            </joint>
+        </ros2_control>
+    </xacro:if>
     <gazebo>
         <plugin filename="ign_ros2_control-system" name="ign_ros2_control::IgnitionROS2ControlPlugin">
             <parameters>$(find snowplow)/config/my_controllers_sim.yaml</parameters>
-            <!-- <controller_manager_name>controller_manager</controller_manager_name> -->
+        </plugin>
+        <plugin name="motor_controller" filename="libsnowplow_motor_controller.so">
+            <parameters>$(find snowplow)/config/my_controllers.yaml</parameters>
         </plugin>
     </gazebo>

Commit message: Adding rtk functionality components

File: src/snowplow/description/gps_ign.xacro (robot description, xacro)
@@ -4,5 +4,5 @@
     <parent link="chassis"/>
     <child link="gps_link"/>
-    <origin xyz="-0.375 0 0.278" rpy="0 0.18 0"/>
+    <origin xyz="-0.375 0.345 0.556" rpy="0 0.18 0"/>
   </joint>
   <link name="gps_link">
