Commit message: Fixing slam and nav2

File: src/nav2_outdoor_example/urdf/lidar_ign.xacro (robot description, xacro)
@@ -3,7 +3,7 @@
     <!-- LIDAR -->
     <joint name="laser_joint" type="fixed">
-        <parent link="chassis"/>
+        <parent link="base_link"/>
         <child link="laser_frame"/>
-        <origin xyz="0.10 0 0.66" rpy="0 0 0"/>
+        <origin xyz="0.10 0 ${-wheel_offset_z + 0.66}" rpy="0 0 0"/>
     </joint>
     <link name="laser_frame">
@@ -39,5 +39,5 @@
     <gazebo reference="laser_frame">
         <material>Gazebo/Black</material>
-        <sensor name="gpu_lidar" type="gpu_lidar">
+        <sensor name="laser_frame" type="gpu_lidar">
             <pose relative_to='laser_frame'> 0 0 0 0 0 4.713 </pose>
             <topic>scan</topic>

Commit message: Fixing lidar rotation

File: src/nav2_outdoor_example/urdf/lidar_ign.xacro (robot description, xacro)
@@ -5,5 +5,5 @@
         <parent link="base_link"/>
         <child link="laser_frame"/>
-        <origin xyz="0.10 0 ${-wheel_offset_z + 0.66}" rpy="0 0 0"/>
+        <origin xyz="0.10 0 ${-wheel_offset_z + 0.66}" rpy="0 0 4.713"/>
     </joint>
     <link name="laser_frame">
@@ -41,5 +41,5 @@
         <sensor name="laser_frame" type="gpu_lidar">
             <ignition_frame_id>laser_frame</ignition_frame_id>
-            <pose relative_to='laser_frame'> 0 0 0 0 0 4.713 </pose>
+            <pose relative_to='laser_frame'> 0 0 0 0 0 0 </pose>
             <topic>scan</topic>
             <visualize>true</visualize>

Commit message: Making lidar 360 instead of 180

File: src/nav2_outdoor_example/urdf/lidar_ign.xacro (robot description, xacro)
@@ -5,5 +5,5 @@
         <parent link="base_link"/>
         <child link="laser_frame"/>
-        <origin xyz="0.10 0 ${-wheel_offset_z + 0.66}" rpy="0 0 0"/>
+        <origin xyz="0.10 0 ${-wheel_offset_z + 0.66}" rpy="0 0 4.713"/>
     </joint>
     <link name="laser_frame">
@@ -40,5 +40,5 @@
         <material>Gazebo/Black</material>
         <sensor name="laser_frame" type="gpu_lidar">
-            <pose relative_to='laser_frame'> 0 0 0 0 0 4.713 </pose>
+            <pose relative_to='laser_frame'> 0 0 0 0 0 0 </pose>
             <topic>scan</topic>
             <visualize>true</visualize>
@@ -48,5 +48,4 @@
                     <horizontal>
                         <samples>360</samples>
-                        <min_angle>0</min_angle>
                         <min_angle>-3.14</min_angle>
                         <max_angle>3.14</max_angle>
